File: afterglow_whitestar_pb_v30/afterglow_whitestar.kicad_pcb (KiCad board)
At the start: 4 copper layers, 81 x 181.4 mm, 147 parts, among them J3 J13_IN_C, J4 J13_OUT_C, J5 J12_IN_R, J6 J12_OUT_R, J7 Conn_02x03_Odd_Even, J8 Conn_01x07_Male, J9 UART, Q1 IRFR5505, Q10 IRFR3910, Q11 IRFR5505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

Commit message: Finalized (?) v3
Connections:
- J9 pad 1: /arduinonano/D1 -> /arduinonano/D0
- J9 pad 3: /arduinonano/D0 -> /arduinonano/D1
Routing:
- net /arduinonano/D0: track 24.6 -> 18.2 mm
- net /arduinonano/D1: track 20.0 -> 21.2 mm
