File: afterglow_whitestar_pb_v30/arduinonano.kicad_sch (KiCad schematic)
At the start: 9 parts, among them J7 Conn_02x03_Odd_Even, J9 UART, U7 ATmega328-A, Y1 16MHz

Commit message: Finalized (?) v3
Connections:
- net D0: now also J9.1 (Pin_1); no longer J9.3 (Pin_3)
- net D1: now also J9.3 (Pin_3); no longer J9.1 (Pin_1)
Changed lines of the file:
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@@
   (junction (at 104.14 34.29) (diameter 0) (color 0 0 0 0)
   )
-  (junction (at 170.18 100.33) (diameter 0) (color 0 0 0 0)
-  )
-  (junction (at 168.91 102.87) (diameter 0) (color 0 0 0 0)
+  (junction (at 170.18 102.87) (diameter 0) (color 0 0 0 0)
   )
   (junction (at 205.74 95.25) (diameter 0) (color 0 0 0 0)
   )
   (junction (at 199.39 74.93) (diameter 0) (color 0 0 0 0)
+  )
+  (junction (at 168.91 100.33) (diameter 0) (color 0 0 0 0)
   )
   (junction (at 104.14 44.45) (diameter 0) (color 0 0 0 0)
@@
     (stroke (width 0) (type default) (color 0 0 0 0))
   )
-  (wire (pts (xy 226.06 121.92) (xy 226.06 125.73))
-    (stroke (width 0) (type default) (color 0 0 0 0))
-  )
   (wire (pts (xy 168.91 64.77) (xy 175.26 64.77))
     (stroke (width 0) (type default) (color 0 0 0 0))
@@
     (stroke (width 0) (type default) (color 0 0 0 0))
   )
-  (wire (pts (xy 170.18 100.33) (xy 171.45 100.33))
+  (wire (pts (xy 167.64 100.33) (xy 168.91 100.33))
     (stroke (width 0) (type default) (color 0 0 0 0))
   )
@@
     (stroke (width 0) (type default) (color 0 0 0 0))
   )
-  (wire (pts (xy 229.87 121.92) (xy 226.06 121.92))
+  (wire (pts (xy 170.18 121.92) (xy 229.87 121.92))
     (stroke (width 0) (type default) (color 0 0 0 0))
   )
@@
     (stroke (width 0) (type default) (color 0 0 0 0))
   )
+  (wire (pts (xy 168.91 127) (xy 168.91 100.33))
+    (stroke (width 0) (type default) (color 0 0 0 0))
+  )
   (wire (pts (xy 167.64 57.15) (xy 175.26 57.15))
     (stroke (width 0) (type default) (color 0 0 0 0))
@@
     (stroke (width 0) (type default) (color 0 0 0 0))
   )
-  (wire (pts (xy 170.18 125.73) (xy 226.06 125.73))
-    (stroke (width 0) (type default) (color 0 0 0 0))
-  )
   (wire (pts (xy 152.4 46.99) (xy 154.94 46.99))
     (stroke (width 0) (type default) (color 0 0 0 0))
@@
     (stroke (width 0) (type default) (color 0 0 0 0))
   )
-  (wire (pts (xy 168.91 102.87) (xy 168.91 127))
-    (stroke (width 0) (type default) (color 0 0 0 0))
-  )
   (wire (pts (xy 196.85 74.93) (xy 199.39 74.93))
     (stroke (width 0) (type default) (color 0 0 0 0))
@@
     (stroke (width 0) (type default) (color 0 0 0 0))
   )
-  (wire (pts (xy 167.64 102.87) (xy 168.91 102.87))
+  (wire (pts (xy 167.64 102.87) (xy 170.18 102.87))
     (stroke (width 0) (type default) (color 0 0 0 0))
   )
@@
     (stroke (width 0) (type default) (color 0 0 0 0))
   )
-  (wire (pts (xy 168.91 102.87) (xy 171.45 102.87))
-    (stroke (width 0) (type default) (color 0 0 0 0))
-  )
   (wire (pts (xy 168.91 64.77) (xy 168.91 78.74))
     (stroke (width 0) (type default) (color 0 0 0 0))
@@
     (stroke (width 0) (type default) (color 0 0 0 0))
   )
-  (wire (pts (xy 167.64 100.33) (xy 170.18 100.33))
-    (stroke (width 0) (type default) (color 0 0 0 0))
-  )
-  (wire (pts (xy 170.18 100.33) (xy 170.18 125.73))
-    (stroke (width 0) (type default) (color 0 0 0 0))
-  )
   (wire (pts (xy 167.64 64.77) (xy 168.91 64.77))
     (stroke (width 0) (type default) (color 0 0 0 0))
@@
     (stroke (width 0) (type default) (color 0 0 0 0))
   )
+  (wire (pts (xy 170.18 102.87) (xy 170.18 121.92))
+    (stroke (width 0) (type default) (color 0 0 0 0))
+  )
   (wire (pts (xy 181.61 66.04) (xy 201.93 66.04))
     (stroke (width 0) (type default) (color 0 0 0 0))
@@
     (stroke (width 0) (type default) (color 0 0 0 0))
   )
+  (wire (pts (xy 168.91 100.33) (xy 171.45 100.33))
+    (stroke (width 0) (type default) (color 0 0 0 0))
+  )
   (wire (pts (xy 152.4 125.73) (xy 152.4 132.08))
     (stroke (width 0) (type default) (color 0 0 0 0))
@@
     (stroke (width 0) (type default) (color 0 0 0 0))
   )
-  (wire (pts (xy 168.91 127) (xy 229.87 127))
-    (stroke (width 0) (type default) (color 0 0 0 0))
-  )
   (wire (pts (xy 170.18 67.31) (xy 175.26 67.31))
     (stroke (width 0) (type default) (color 0 0 0 0))
@@
     (stroke (width 0) (type default) (color 0 0 0 0))
   )
+  (wire (pts (xy 170.18 102.87) (xy 171.45 102.87))
+    (stroke (width 0) (type default) (color 0 0 0 0))
+  )
   (wire (pts (xy 237.49 111.76) (xy 240.03 111.76))
     (stroke (width 0) (type default) (color 0 0 0 0))
@@
     (stroke (width 0) (type default) (color 0 0 0 0))
   )
+  (wire (pts (xy 229.87 127) (xy 168.91 127))
+    (stroke (width 0) (type default) (color 0 0 0 0))
+  )
